File: Eagle_Files/Automated_Blinds_Remote.brd (EAGLE design)
At the start: 160 x 100 mm, 25 parts, among them U1 LPC1114FN28/102, U2 UA78MC

Commit message: Finished PCB design for remote control
Parts:
- added R8, R9: 10, rcl:0207/10
- moved UART 102.3 mm to (27.9, 5.08), turned to 180 degrees
- moved R6 29.5 mm to (80.0, 39.4), turned to 90 degrees
- moved JTAG/SWD1 29.2 mm to (67.3, 10.2)
- moved BACK_BUTTON 18.9 mm to (102.9, 29.2), turned to 180 degrees
- moved R4 15.3 mm to (137.2, 27.9)
- moved C1 12.0 mm to (27.9, 33.0), turned to 270 degrees
- moved ENTER_BUTTON 10.2 mm to (108.0, 78.7), turned to 0 degrees
- moved R5 9.25 mm to (87.6, 76.2)
- moved C2 8.52 mm to (39.4, 33.0), turned to 270 degrees
- moved U1 5.68 mm to (53.3, 55.9), turned to 180 degrees
- moved LEFT_BUTTON 5.08 mm to (129.5, 36.8)
- moved RIGHT_BUTTON 3.81 mm to (129.5, 67.3), turned to 180 degrees
- moved C3 2.54 mm to (17.8, 78.7)
- moved R2 2.54 mm to (101.6, 44.5)
- moved R3 1.80 mm to (106.7, 64.8)
Connections:
- net +3V3: now also R8.2, R9.2
- net N$1: now also R8.1, R9.1
Routing:
- net GND: track 50.8 -> 618.9 mm
- net +3V3: track 36.2 -> 362.3 mm, vias 0 -> 3
- net SWDIO: track 0.00 -> 152.4 mm, vias 0 -> 2
- net BACK_B: track 0.00 -> 127.4 mm
- net DOWN_B: track 0.00 -> 119.3 mm
- net LEFT_B: track 0.00 -> 103.7 mm
- net RIGHT_B: track 0.00 -> 89.1 mm
- net SCL: track 0.00 -> 78.7 mm, vias 0 -> 2
- net SCREEN_RST: track 0.00 -> 78.7 mm, vias 0 -> 1
- net SWCLK: track 0.00 -> 76.2 mm, vias 0 -> 2
- net ENTER_B: track 0.00 -> 59.9 mm
- net IR_CONTROL: track 0.00 -> 57.2 mm, vias 0 -> 1
- net UP_B: track 0.00 -> 54.0 mm
- net TX: track 0.00 -> 46.3 mm
- net RX: track 0.00 -> 46.3 mm
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
Commit message: Updated value of button pull-ups in schematic
Parts:
- R1, R2, R3, R4, R5, R6: value 1K -> 10K
Changed lines of the file:
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@@
 <element name="OLED" library="pinhead" package="1X06" value="" x="8.89" y="31.75" rot="R270"/>
 <element name="PWR" library="pinhead" package="1X03" value="" x="53.34" y="95.25"/>
-<element name="R1" library="rcl" package="0207/10" value="1K" x="92.71" y="55.88" rot="R180"/>
-<element name="R2" library="rcl" package="0207/10" value="1K" x="101.6" y="44.45" rot="R180"/>
-<element name="R3" library="rcl" package="0207/10" value="1K" x="106.68" y="64.77" rot="R180"/>
-<element name="R4" library="rcl" package="0207/10" value="1K" x="137.16" y="27.94"/>
-<element name="R5" library="rcl" package="0207/10" value="1K" x="87.63" y="76.2" rot="R180"/>
-<element name="R6" library="rcl" package="0207/10" value="1K" x="80.01" y="39.37" rot="R90"/>
+<element name="R1" library="rcl" package="0207/10" value="10K" x="92.71" y="55.88" rot="R180"/>
+<element name="R2" library="rcl" package="0207/10" value="10K" x="101.6" y="44.45" rot="R180"/>
+<element name="R3" library="rcl" package="0207/10" value="10K" x="106.68" y="64.77" rot="R180"/>
+<element name="R4" library="rcl" package="0207/10" value="10K" x="137.16" y="27.94"/>
+<element name="R5" library="rcl" package="0207/10" value="10K" x="87.63" y="76.2" rot="R180"/>
+<element name="R6" library="rcl" package="0207/10" value="10K" x="80.01" y="39.37" rot="R90"/>
 <element name="R7" library="rcl" package="0207/10" value="10" x="10.16" y="66.04"/>
 <element name="RIGHT_BUTTON" library="B3F-1000" package="SW_B3F-1000" value="B3F-1000" x="129.54" y="67.31" rot="R180">
